Commit message: phoenix launch option

File: packages/simulation/phoenix_sim_description/urdf/macros.xacro (robot description, xacro)
@@ -43,8 +43,8 @@
     </xacro:macro>
     <xacro:macro name="robot_wheel">
-        <mesh filename="package://ezrassor_sim_description/meshes/wheel.dae" scale="0.35 0.35 0.35"></mesh>
+        <mesh filename="package://phoenix_sim_description/meshes/wheel.dae" scale="0.35 0.35 0.35"></mesh>
     </xacro:macro>
     <xacro:macro name="base_unit">
-        <mesh filename="package://ezrassor_sim_description/meshes/base_unit.dae" scale="0.35 0.35 0.35"></mesh>
+        <mesh filename="package://phoenix_sim_description/meshes/base_unit.dae" scale="0.35 0.35 0.35"></mesh>
     </xacro:macro>
     <xacro:macro name="drum_arm">

File: packages/simulation/phoenix_sim_description/urdf/phoenix.xacro (robot description, xacro)
@@ -3,7 +3,7 @@
   <xacro:property name="cameraSize" value="0.01"/>
   <xacro:property name="cameraMass" value="0.1"/>
-  <xacro:include filename="$(find ezrassor_sim_description)/urdf/ezrassor.gazebo" />
-  <xacro:include filename="$(find ezrassor_sim_description)/urdf/materials.xacro" />
-  <xacro:include filename="$(find ezrassor_sim_description)/urdf/macros.xacro" />
+  <xacro:include filename="$(find phoenix_sim_description)/urdf/phoenix.gazebo" />
+  <xacro:include filename="$(find phoenix_sim_description)/urdf/materials.xacro" />
+  <xacro:include filename="$(find phoenix_sim_description)/urdf/macros.xacro" />
   <!--Below are all of the robot's Links/-->
   <link name='base_link'>
